File: smart_helmet.kicad_pcb (KiCad board)
At the start: 2 copper layers, 62.3 x 62.3 mm, 3 parts, among them U1 MQ-6, U2 ATmega32A-A

Commit message: initial commit
Parts:
- moved BZ1 18.2 mm to (182.7, 86.5)
- moved U1 18.2 mm to (165.4, 53.6)
- moved U2 18.2 mm to (152.1, 85.3)
Routing:
- net GND: track 164.0 -> 358.0 mm
- net +5V: track 234.4 -> 359.8 mm
- net Net-(U1-A2): track 40.1 -> 73.9 mm
- net Net-(U1-B2): track 69.3 -> 93.2 mm
Other:
- board size 62.3 x 62.3 mm -> 61.5 x 55 mm
